Commit message: Joint wobble fixed by adjusting pid values

File: hex_bot_description/macros/make_servo.xacro (robot description, xacro)
@@ -8,4 +8,5 @@
   <xacro:macro name="make_servo_with_origin" params="name len wid hei mas parent *origin">
     <xacro:make_box_with_origin name="${name}" len="${len}" wid="${wid}" hei="${hei}" mas="${mas}">
+      <!-- The servo's origin is set at the front half -->
       <origin xyz="${-servo_len/2} 0 0" rpy="0 0 0"/>
     </xacro:make_box_with_origin>

File: hex_bot_description/urdf/config.xacro (robot description, xacro)
@@ -5,5 +5,5 @@
   <xacro:property name="body_wid" value="0.10"/>
   <xacro:property name="body_hei" value="0.05"/>
-  <xacro:property name="body_mas" value="0.90"/>
+  <xacro:property name="body_mas" value="0.50"/>
   <xacro:property name="servo_len" value="0.025"/>
   <xacro:property name="servo_wid" value="0.015"/>
@@ -16,8 +16,8 @@
   <xacro:property name="femur_wid" value="0.010"/>
   <xacro:property name="femur_hei" value="0.015"/>
-  <xacro:property name="femur_mas" value="0.100"/>
+  <xacro:property name="femur_mas" value="0.150"/>
   <xacro:property name="tibia_len" value="0.070"/>
   <xacro:property name="tibia_wid" value="0.010"/>
   <xacro:property name="tibia_hei" value="0.015"/>
-  <xacro:property name="tibia_mas" value="0.100"/>
+  <xacro:property name="tibia_mas" value="0.150"/>
 </robot>
