Commit message: Six feet and controllers added.

File: hex_bot_description/macros/make_leg.xacro (robot description, xacro)
@@ -2,7 +2,7 @@
 <!-- Macro to build a leg -->
 <robot name="hex_bot" xmlns:xacro="http://www.ros.org/wiki/xacro">
-  <xacro:macro name="make_leg" params="prefix parent">
+  <xacro:macro name="make_leg" params="prefix parent *origin">
     <xacro:make_servo_with_origin name="${prefix}_servo_1" len="${servo_len}" wid="${servo_wid}" hei="${servo_hei}" mas="${servo_mas}" parent="${parent}">
-      <origin xyz="0.05 0.06 0" rpy="0 0 -1.57"/>
+      <insert_block name="origin"/>
     </xacro:make_servo_with_origin>
     <xacro:make_servo_with_origin name="${prefix}_servo_2" len="${servo_len}" wid="${servo_wid}" hei="${servo_hei}" mas="${servo_mas}" parent="${prefix}_servo_1">

File: hex_bot_description/urdf/hex_bot.xacro (robot description, xacro)
@@ -9,5 +9,22 @@
   <link name="base_link"/>
   <xacro:make_box name="body" len="${body_len}" wid="${body_wid}" hei="${body_hei}" mas="${body_mas}"/>
-  <xacro:make_leg prefix="LEG" parent="body"/>
+  <xacro:make_leg prefix="FL" parent="body">
+    <origin xyz="0.05 0.06 0" rpy="0 0 -1.57"/>
+  </xacro:make_leg>
+  <xacro:make_leg prefix="FR" parent="body">
+    <origin xyz="0.05 -0.06 0" rpy="0 0 1.57"/>
+  </xacro:make_leg>
+  <xacro:make_leg prefix="ML" parent="body">
+    <origin xyz="0.00 0.06 0" rpy="0 0 -1.57"/>
+  </xacro:make_leg>
+  <xacro:make_leg prefix="MR" parent="body">
+    <origin xyz="0.00 -0.06 0" rpy="0 0 1.57"/>
+  </xacro:make_leg>
+  <xacro:make_leg prefix="BL" parent="body">
+    <origin xyz="-0.05 0.06 0" rpy="0 0 -1.57"/>
+  </xacro:make_leg>
+  <xacro:make_leg prefix="BR" parent="body">
+    <origin xyz="-0.05 -0.06 0" rpy="0 0 1.57"/>
+  </xacro:make_leg>
   <xacro:make_fixed_joint child="body" parent="base_link"/>
 </robot>
